File: forager-pcb/forager-pcb.kicad_pcb (KiCad board)
At the start: 2 copper layers, 236.5 x 96.3 mm, 90 parts, among them J1 Conn_01x02_Pin, J2 Conn_01x02_Pin

Commit message: add a power switch, change the battery test points to through hole
Parts:
- removed TP1, TP2, TP3, TP4: TestPoint, TestPoint:TestPoint_Pad_D2.0mm
- added J3: Conn_01x02_Pin, Connector_PinHeader_2.54mm:PinHeader_1x02_P2.54mm_Vertical, B.Cu at (-98.0, 7.25)
- added J4: Conn_01x02_Pin, Connector_PinHeader_2.54mm:PinHeader_1x02_P2.54mm_Vertical, B.Cu at (98.0, 3.46)
- added PSW1: SW_SPDT, PCM_marbastlib-various:SW_MSK12C02-HB, B.Cu at (-116.5, -16.0)
- added PSW2: SW_SPDT, PCM_marbastlib-various:SW_MSK12C02-HB, B.Cu at (116.5, -16.0)
Connections:
- J1 pad 1: LBAT -> LBAT_CONN
- J2 pad 1: RBAT -> RBAT_CONN
Routing:
- net RBAT: track 83.9 -> 26.1 mm, vias 0 -> 1
- net LBAT: track 90.7 -> 37.6 mm, vias 0 -> 2
- net LBAT_CONN: track 0.00 -> 40.2 mm
- net /LROW3: track 159.1 -> 122.3 mm, vias 0 -> 2
- net RBAT_CONN: track 0.00 -> 36.4 mm, vias 0 -> 1
- net /LROW1: track 136.9 -> 103.5 mm, vias 0 -> 2
- net /LROW2: track 84.9 -> 87.4 mm
- net /RCOL0: track 53.5 -> 51.6 mm
- net /RROW3: track 110.5 -> 112.1 mm, vias 0 -> 2
- net /RCOL1: track 67.4 -> 65.9 mm
- net /RROW2: track 113.4 -> 111.9 mm, vias 0 -> 2
- net Net-(LD7-A): track 66.7 -> 67.8 mm
- net /LCOL3: track 133.6 -> 132.8 mm
- net Net-(LD6-A): track 91.4 -> 92.0 mm
- net /LCOL1: track 82.1 -> 81.6 mm
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Other:
- board text added: "Negative Positive"
- board text added: "Positive Negative"
- board text removed: "+"

Commit message: update revision number to 2.1
Other:
- board text added: "rev. 2.1"
- board text removed: "rev. 2"
